File: PCB/001.kicad_pcb (KiCad board)
At the start: 2 copper layers, 69.4 x 98.2 mm, 41 parts

Commit message: Add HoleBig
Parts:
- added REF**: Hole_Big, ArduinoBadge:Hole_Big, F.Cu at (133.3, 68.3)
- moved REF** 3.07 mm to (133.3, 77.3)
- moved REF** 3.07 mm to (133.3, 97.6)
Changed lines of the file:
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@@
-(kicad_pcb (version 20171130) (host pcbnew 6.0.0-rc1-unknown-59b0f55~66~ubuntu16.04.1)
+(kicad_pcb (version 20171130) (host pcbnew 6.0.0-rc1-unknown-5b3202d~66~ubuntu16.04.1)
   (general
     (thickness 1.6)
@@
     (tracks 0)
     (zones 0)
-    (modules 41)
+    (modules 42)
     (nets 1)
   )
@@
   )
   (module Connector_PinSocket_2.54mm:PinSocket_1x14_P2.54mm_Vertical_SMD_Pin1Right (layer B.Cu)
-    (at 132.715 74.268496 270)
+    (at 133.2738 77.291096 270)
     (descr "surface-mounted straight socket strip, 1x14, 2.54mm pitch, single row, style 2 (pin 1 right) (https://cdn.harwin.com/pdfs/M20-786.pdf), script generated")
     (tags "Surface mounted socket strip SMD 1x14 2.54mm single row style2 pin1 right")
     (attr smd)
-    (fp_text reference REF** (at 0 19.38 270) (layer B.SilkS)
+    (fp_text reference REF** (at 5.690704 16.4338 270) (layer B.Fab)
       (effects (font (size 1 1) (thickness 0.15)) (justify mirror))
     )
@@
   )
   (module Connector_PinSocket_2.54mm:PinSocket_1x14_P2.54mm_Vertical_SMD_Pin1Right (layer B.Cu)
-    (at 132.715 94.588496 270)
+    (at 133.2738 97.611096 270)
     (descr "surface-mounted straight socket strip, 1x14, 2.54mm pitch, single row, style 2 (pin 1 right) (https://cdn.harwin.com/pdfs/M20-786.pdf), script generated")
     (tags "Surface mounted socket strip SMD 1x14 2.54mm single row style2 pin1 right")
     (attr smd)
-    (fp_text reference REF** (at 0 19.38 270) (layer B.SilkS)
+    (fp_text reference REF** (at -5.891696 16.5354 270) (layer B.Fab)
       (effects (font (size 1 1) (thickness 0.15)) (justify mirror))
     )
@@
       (xy 0.32762 -1.356294) (xy 0.334747 -1.354539)) (layer F.Mask) (width 0.38324))
   )
+  (module ArduinoBadge:Hole_Big (layer F.Cu)
+    (at 133.35 68.2752)
+    (fp_text reference REF** (at 0 0.5) (layer F.SilkS)
+      (effects (font (size 1 1) (thickness 0.15)))
+    )
+    (fp_text value Hole_Big (at 0 -0.5) (layer F.Fab)
+      (effects (font (size 1 1) (thickness 0.15)))
+    )
+    (pad 1 thru_hole roundrect (at 0 0) (size 15 7) (drill oval 14 6) (layers *.Cu *.Mask) (roundrect_rratio 0.25))
+  )
   (gr_circle (center 117.348 76.962) (end 118.618 76.962) (layer Dwgs.User) (width 0.15))

Commit message: Update Edge
Parts:
- removed the REF** at (133.3, 68.3)
- removed the svg2mod at (133.3, 111.1)
- added svg2mod: G***, ArduinoBadge:Edge.SilkS.04.4, F.Cu at (133.3, 110.7)
- added svg2mod: G***, ArduinoBadge:Edge.Back.Only.SilkS.02, B.Cu at (133.5, 110.8)
- added svg2mod: G***, ArduinoBadge:Edge.Only.SilkS.02, F.Cu at (133.3, 110.7)
- added svg2mod: G***, ArduinoBadge:Fig.02.Cu.Mask, F.Cu at (147.9, 78.2)
- added svg2mod: G***, ArduinoBadge:Fig.01.Cu.Mask, F.Cu at (102.7, 83.3)
- added svg2mod: G***, ArduinoBadge:Holder.Cu.Mask.01, B.Cu at (133.4, 67.3)
- added svg2mod: G***, ArduinoBadge:Holder.Cu.Mask.01, F.Cu at (133.0, 67.3)
- moved svg2mod 11.1 mm to (114.9, 142.8)
- moved svg2mod 9.06 mm to (133.4, 129.3)
- moved svg2mod 6.02 mm to (158.9, 102.7)
- moved svg2mod 2.44 mm to (154.7, 150.8)
Other:
- board size 69.4 x 98.2 mm -> 75 x 98.8 mm
