File: 001/001.sch (KiCad schematic (older format))
At the start: 24 parts, among them J1 Conn_01x02_Female, J10 Conn_01x02_Female, J11 Conn_01x02_Female, J12 Conn_01x02_Female, J13 Conn_01x02_Female, J14 Conn_01x02_Female, J15 Conn_01x02_Female, J16 Conn_01x02_Female, J2 Conn_01x02_Female, J3 Conn_01x02_Female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

Commit message: Update
Parts:
- added J17, J18: Conn_01x14, symbol Connector_Generic:Conn_01x14
Connections:
- net GND: now also J18.4 (Pin_4)
- net VCC: no longer J1.1 (Pin_1), U1.1 (VCC)
- net ~2: now reaches J1.2 (Pin_2), U1.2 (IN)
- net ~2: now also J17.11 (Pin_11)
- new net +3V3: J1.1 (Pin_1), J18.3 (Pin_3), U1.1 (VCC)
- new net +5V: J18.1 (Pin_1)
- new net 1: J17.10 (Pin_10)
- new net 10-MISO: J18.10 (Pin_10)
- new net 11-SDA: J18.9 (Pin_9)
- new net 12-SCL: J18.8 (Pin_8)
- new net 13->RX: J18.7 (Pin_7)
- new net 14<-TX: J18.6 (Pin_6)
- new net 6: J18.14 (Pin_14)
- new net 7: J18.13 (Pin_13)
- new net 8-MOSI: J18.12 (Pin_12)
- new net 9-SCK: J18.11 (Pin_11)
- new net A1: J17.3 (Pin_3)
- new net A2: J17.4 (Pin_4)
- new net A3: J17.5 (Pin_5)
- new net A4: J17.6 (Pin_6)
- new net A5: J17.7 (Pin_7)
- new net A6: J17.8 (Pin_8)
- new net AREF: J17.1 (Pin_1)
- new net DAC0-A0: J17.2 (Pin_2)
- new net RESET: J18.5 (Pin_5)
- new net VIN: J18.2 (Pin_2)
- new net ~3: J17.12 (Pin_12)
- new net ~4: J17.13 (Pin_13)
- new net ~5: J17.14 (Pin_14)

Commit message: Update H
Parts:
- J17, J18: footprint (none) -> Connector_PinSocket_2.54mm:PinSocket_1x14_P2.54mm_Vertical_SMD_Pin1Left
Changed lines of the file:
@@
 F 0 "J17" H 6150 4700 50  0000 L CNN
 F 1 "Conn_01x14" H 6280 3901 50  0001 L CNN
-F 2 "" H 6200 4000 50  0001 C CNN
+F 2 "Connector_PinSocket_2.54mm:PinSocket_1x14_P2.54mm_Vertical_SMD_Pin1Left" H 6200 4000 50  0001 C CNN
 F 3 "~" H 6200 4000 50  0001 C CNN
 	1    6200 4000
@@
 F 0 "J18" H 6950 4700 50  0000 L CNN
 F 1 "Conn_01x14" H 7080 3901 50  0001 L CNN
-F 2 "" H 7000 4000 50  0001 C CNN
+F 2 "Connector_PinSocket_2.54mm:PinSocket_1x14_P2.54mm_Vertical_SMD_Pin1Left" H 7000 4000 50  0001 C CNN
 F 3 "~" H 7000 4000 50  0001 C CNN
 	1    7000 4000

Commit message: Add new shapes
Parts:
- J1, J10, J11, J12, J13, J14, J15, J16, J2, J3, J4, J5, J6, J7, J8, J9: symbol Connector:Conn_01x02_Female -> 001-rescue:Conn_01x02_Female-Connector
- J17, J18: symbol Connector_Generic:Conn_01x14 -> 001-rescue:Conn_01x14-Connector_Generic
Changed lines of the file:
@@
 $EndDescr
 $Comp
-L Connector:Conn_01x02_Female J2
+L 001-rescue:Conn_01x02_Female-Connector J2
 U 1 1 5C4A7885
 P 2250 2250
@@
 $EndComp
 $Comp
-L Connector:Conn_01x02_Female J1
+L 001-rescue:Conn_01x02_Female-Connector J1
 U 1 1 5C4A796D
 P 1000 2250
@@
 $EndComp
 $Comp
-L Connector:Conn_01x02_Female J6
+L 001-rescue:Conn_01x02_Female-Connector J6
 U 1 1 5C4BEE00
 P 2250 2950
@@
 $EndComp
 $Comp
-L Connector:Conn_01x02_Female J3
+L 001-rescue:Conn_01x02_Female-Connector J3
 U 1 1 5C4BEE0A
 P 1000 2950
@@
 	1275 3050 1200 3050
 $Comp
-L Connector:Conn_01x02_Female J7
+L 001-rescue:Conn_01x02_Female-Connector J7
 U 1 1 5C4CB9B4
 P 2250 3750
@@
 $EndComp
 $Comp
-L Connector:Conn_01x02_Female J4
+L 001-rescue:Conn_01x02_Female-Connector J4
 U 1 1 5C4CB9BE
 P 1000 3750
@@
 	2000 3750 1925 3750
 $Comp
-L Connector:Conn_01x02_Female J8
+L 001-rescue:Conn_01x02_Female-Connector J8
 U 1 1 5C4D08E8
 P 2250 4425
@@
 $EndComp
 $Comp
-L Connector:Conn_01x02_Female J5
+L 001-rescue:Conn_01x02_Female-Connector J5
 U 1 1 5C4D08F2
 P 1000 4425
@@
 	1275 4525 1200 4525
 $Comp
-L Connector:Conn_01x02_Female J13
+L 001-rescue:Conn_01x02_Female-Connector J13
 U 1 1 5C4E30D8
 P 3750 2250
@@
 $EndComp
 $Comp
-L Connector:Conn_01x02_Female J9
+L 001-rescue:Conn_01x02_Female-Connector J9
 U 1 1 5C4E30E2
 P 2500 2250
@@
 $EndComp
 $Comp
-L Connector:Conn_01x02_Female J14
+L 001-rescue:Conn_01x02_Female-Connector J14
 U 1 1 5C4E3114
 P 3750 2950
@@
 $EndComp
 $Comp
-L Connector:Conn_01x02_Female J10
+L 001-rescue:Conn_01x02_Female-Connector J10
 U 1 1 5C4E311E
 P 2500 2950
@@
 	2775 3050 2700 3050
 $Comp
-L Connector:Conn_01x02_Female J15
+L 001-rescue:Conn_01x02_Female-Connector J15
 U 1 1 5C4E3158
 P 3750 3750
@@
 $EndComp
 $Comp
-L Connector:Conn_01x02_Female J11
+L 001-rescue:Conn_01x02_Female-Connector J11
 U 1 1 5C4E3162
 P 2500 3750
@@
 	3500 3750 3425 3750
 $Comp
-L Connector:Conn_01x02_Female J16
+L 001-rescue:Conn_01x02_Female-Connector J16
 U 1 1 5C4E3198
 P 3750 4425
@@
 $EndComp
 $Comp
-L Connector:Conn_01x02_Female J12
+L 001-rescue:Conn_01x02_Female-Connector J12
 U 1 1 5C4E31A2
 P 2500 4425
@@
 	2775 3850 2700 3850
 $Comp
-L Connector_Generic:Conn_01x14 J17
+L 001-rescue:Conn_01x14-Connector_Generic J17
 U 1 1 5C4D1F80
 P 6200 4000
@@
 $EndComp
 $Comp
-L Connector_Generic:Conn_01x14 J18
+L 001-rescue:Conn_01x14-Connector_Generic J18
 U 1 1 5C4D6F4B
 P 7000 4000
@@
 $EndComp
 $Comp
-L power:VIN #PWR010
+L 001-rescue:VIN-power #PWR010
 U 1 1 5C55DEFA
 P 7325 3500
@@
 $EndComp
 $Comp
-L power:VIN #PWR014
+L 001-rescue:VIN-power #PWR014
 U 1 1 5C566CBC
 P 9425 1000
