File: 004/001.sch (KiCad schematic (older format))
At the start: 37 parts, among them J1 CONN_01X08, J2 CONN_01X08, U1 2019.All.Mask.02, U10 Holder.Cu.Mask.01, U11 logo.B.Mask.Der.01, U12 logo.B.Mask.Izq.01, U13 logo.F.Mask.Der.01, U14 logo.F.Mask.Izq.01, U15 MKR_Family, U2 2019.All.Mask.03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

Commit message: Rooteo
Se rooteo la carpeta 004 coin dos versiones una a una capa y la otra en las dos, saludos! @antonio_raptors
Parts:
- D1, D10, D2, D3, D4, D5, D6, D7, D8, D9: symbol device:LED_ALT -> 001-rescue:LED_ALT-device
- J1, J2: symbol conn:CONN_01X08 -> 001-rescue:CONN_01X08-conn
- R1, R10, R2, R3, R4, R5, R6, R7, R8, R9: symbol device:R -> 001-rescue:R-device
Changed lines of the file:
@@
 EESchema Schematic File Version 4
 LIBS:001-cache
-EELAYER 29 0
+EELAYER 26 0
 EELAYER END
 $Descr USLetter 11000 8500
@@
 	9850 1125 9850 1000
 $Comp
-L device:LED_ALT D1
+L 001-rescue:LED_ALT-device D1
 U 1 1 5C5AB63A
 P 1450 775
@@
 $EndComp
 $Comp
-L device:R R1
+L 001-rescue:R-device R1
 U 1 1 5C5AC812
 P 1025 775
@@
 $EndComp
 $Comp
-L device:LED_ALT D2
+L 001-rescue:LED_ALT-device D2
 U 1 1 5C5B1608
 P 1450 1275
@@
 $EndComp
 $Comp
-L device:R R2
+L 001-rescue:R-device R2
 U 1 1 5C5B1612
 P 1025 1275
@@
 $EndComp
 $Comp
-L device:LED_ALT D3
+L 001-rescue:LED_ALT-device D3
 U 1 1 5C5B593B
 P 1450 1775
@@
 $EndComp
 $Comp
-L device:R R3
+L 001-rescue:R-device R3
 U 1 1 5C5B5945
 P 1025 1775
@@
 $EndComp
 $Comp
-L device:LED_ALT D4
+L 001-rescue:LED_ALT-device D4
 U 1 1 5C5B595C
 P 1450 2275
@@
 $EndComp
 $Comp
-L device:R R4
+L 001-rescue:R-device R4
 U 1 1 5C5B5966
 P 1025 2275
@@
 $EndComp
 $Comp
-L device:LED_ALT D5
+L 001-rescue:LED_ALT-device D5
 U 1 1 5C5B8FE3
 P 1450 2775
@@
 $EndComp
 $Comp
-L device:R R5
+L 001-rescue:R-device R5
 U 1 1 5C5B8FED
 P 1025 2775
@@
 $EndComp
 $Comp
-L device:LED_ALT D6
+L 001-rescue:LED_ALT-device D6
 U 1 1 5C5B9004
 P 1450 3275
@@
 $EndComp
 $Comp
-L device:R R6
+L 001-rescue:R-device R6
 U 1 1 5C5B900E
 P 1025 3275
@@
 $EndComp
 $Comp
-L device:LED_ALT D7
+L 001-rescue:LED_ALT-device D7
 U 1 1 5C5B9025
 P 1450 3775
@@
 $EndComp
 $Comp
-L device:R R7
+L 001-rescue:R-device R7
 U 1 1 5C5B902F
 P 1025 3775
@@
 $EndComp
 $Comp
-L device:LED_ALT D8
+L 001-rescue:LED_ALT-device D8
 U 1 1 5C5B9046
 P 1450 4275
@@
 $EndComp
 $Comp
-L device:R R8
+L 001-rescue:R-device R8
 U 1 1 5C5B9050
 P 1025 4275
@@
 	4675 5350 4550 5350
 $Comp
-L conn:CONN_01X08 J1
+L 001-rescue:CONN_01X08-conn J1
 U 1 1 5C5F5D0A
 P 4875 5100
@@
 	4675 5450 4550 5450
 $Comp
-L conn:CONN_01X08 J2
+L 001-rescue:CONN_01X08-conn J2
 U 1 1 5C5F9C11
 P 5475 5100
@@
 NoConn ~ 4575 1700
 $Comp
-L device:LED_ALT D9
+L 001-rescue:LED_ALT-device D9
 U 1 1 5C657D44
 P 1450 4775
@@
 $EndComp
 $Comp
-L device:R R9
+L 001-rescue:R-device R9
 U 1 1 5C657D4E
 P 1025 4775
@@
 $EndComp
 $Comp
-L device:LED_ALT D10
+L 001-rescue:LED_ALT-device D10
 U 1 1 5C657D65
 P 1450 5275
@@
 $EndComp
 $Comp
-L device:R R10
+L 001-rescue:R-device R10
 U 1 1 5C657D6F
 P 1025 5275
